File: PCB/ControlBoard/ControlBoard.sch (KiCad schematic (older format))
At the start: 44 parts, among them J1 LINK-A, J11 ICSPDAT/VO, J2 LINK-B, J3 ICSP, J4 Conn_01x04, J5 PortA, J6 PortB, J7 PortC, J8 Conn_01x08, J9 Conn_01x08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

Commit message: Correct missing symbol in control board schematic.
Parts:
- J2: symbol Custom:AudioJack4_SwitchTR1 -> KTANE:AudioJack4_SwitchTR1
Changed lines of the file:
@@
 $EndComp
 $Comp
-L Custom:AudioJack4_SwitchTR1 J2
+L KTANE:AudioJack4_SwitchTR1 J2
 U 1 1 6086A0F3
 P 10600 2150
