File: PCB/ControlBoard/can.kicad_sch (KiCad schematic)
At the start: 4 parts, among them U5 MCP2562-E-SN

Commit message: First pass of PCB rework.
Parts:
- C12, C8: footprint Capacitor_SMD:C_0805_2012Metric -> Capacitor_SMD:C_0603_1608Metric
Connections:
- net CANH: now also D4.1 (K); no longer D4.2 (K)
- net CANL: now also D4.2 (K); no longer D4.1 (K)
Changed lines of the file:
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@@
     (effects (font (size 1.27 1.27)) (justify left bottom))
   )
-  (global_label "CANL" (shape input) (at 93.98 30.48 180) (fields_autoplaced)
+  (global_label "CANL" (shape input) (at 99.06 30.48 0) (fields_autoplaced)
+    (effects (font (size 1.27 1.27)) (justify left))
+    (property "Intersheetrefs" "${INTERSHEET_REFS}" (at 106.1082 30.48 0)
+      (effects (font (size 1.27 1.27)) (justify left) hide)
+    )
+  )
+  (global_label "CANH" (shape input) (at 93.98 30.48 180) (fields_autoplaced)
     (effects (font (size 1.27 1.27)) (justify right))
-    (property "Intersheetrefs" "${INTERSHEET_REFS}" (at 86.9318 30.48 0)
+    (property "Intersheetrefs" "${INTERSHEET_REFS}" (at 86.6294 30.48 0)
       (effects (font (size 1.27 1.27)) (justify right) hide)
-    )
-  )
-  (global_label "CANH" (shape input) (at 99.06 30.48 0) (fields_autoplaced)
-    (effects (font (size 1.27 1.27)) (justify left))
-    (property "Intersheetrefs" "${INTERSHEET_REFS}" (at 106.4106 30.48 0)
-      (effects (font (size 1.27 1.27)) (justify left) hide)
     )
   )
@@
       (effects (font (size 1.27 1.27)) (justify left))
     )
-    (property "Footprint" "Capacitor_SMD:C_0805_2012Metric" (at 19.05 30.48 0)
+    (property "Footprint" "Capacitor_SMD:C_0603_1608Metric" (at 19.05 30.48 0)
       (effects (font (size 1.27 1.27)) hide)
     )
@@
       (effects (font (size 1.27 1.27)) (justify left))
     )
-    (property "Footprint" "Capacitor_SMD:C_0805_2012Metric" (at 19.05 53.34 0)
-      (effects (font (size 1.27 1.27)) hide)
-    )
+    (property "Footprint" "Capacitor_SMD:C_0603_1608Metric" (at 19.05 53.34 0)
+      (effects (font (size 1.27 1.27)) hide)
+    )

Commit message: ControlBoard B02, with buck regulator fix.
Parts:
- U3: renamed from U5; footprint Package_SO:SOIC-8_3.9x4.9mm_P1.27mm -> Package_DFN_QFN:DFN-8-1EP_3x3mm_P0.65mm_EP1.55x2.4mm; symbol Interface_CAN_LIN:MCP2562-E-SN -> Interface_CAN_LIN:MCP2562-E-MF
- renumbered C8 to C7, C12 to C8, D4 to D10
Connections:
- net CANH: now also D10.2 (K); no longer D10.1 (K)
- net CANL: now also D10.1 (K); no longer D10.2 (K)
- net GND: now also U3.9 (PAD)
