File: PCB/Modules/Keymatrix/Keymatrix.kicad_sch (KiCad schematic)
At the start: 20 parts, among them J1 Matrix1, J2 Matrix2, J3 In, U1 SP720ABTG

Commit message: Upgrade KiCad files from 6.0 to 7.0.
Parts:
- D1, D10, D11, D12, D13, D14, D15, D16, D2, D3, D4, D5, D6, D7, D8, D9: footprint Diode_SMD:D_SOD-123F -> Diode_THT:D_DO-35_SOD27_P7.62mm_Horizontal

Commit message: First pass of PCB rework.
Parts:
- added H1: MountingHole, MountingHole:MountingHole_3.2mm_M3, symbol Mechanical:MountingHole
- D1, D10, D11, D12, D13, D14, D15, D16, D2, D3, D4, D5, D6, D7, D8, D9: footprint Diode_THT:D_DO-35_SOD27_P7.62mm_Horizontal -> Diode_SMD:D_SOD-123F
- J3: footprint Custom:PinHeader_2x08_P2.54mm_Vertical-Centered -> KTANE:PinHeader_2x08_P2.54mm_Vertical-Centered
Connections:
- net +5V: now also J3.2 (Pin_2); no longer J3.11 (Pin_11), J3.13 (Pin_13), J3.15 (Pin_15), J3.9 (Pin_9), U1.16 (V+)
- net COL0: now also J3.1 (Pin_1); no longer J3.16 (Pin_16)
- net COL1: now also J3.3 (Pin_3); no longer J3.14 (Pin_14)
- net COL2: now also J3.5 (Pin_5); no longer J3.12 (Pin_12)
- net COL3: now also J3.7 (Pin_7); no longer J3.10 (Pin_10)
- net GND: now also J3.16 (Pin_16); no longer J3.1 (Pin_1), J3.3 (Pin_3), J3.5 (Pin_5), J3.7 (Pin_7)
- net ROW0: now also D13.1 (K), D5.1 (K), J3.9 (Pin_9); no longer D10.1 (K), D2.1 (K), J3.8 (Pin_8)
- net ROW1: now also D10.1 (K), D14.1 (K), D2.1 (K), D6.1 (K), J3.11 (Pin_11); no longer D11.1 (K), D12.1 (K), D3.1 (K), D4.1 (K), J3.6 (Pin_6)
- net ROW2: now also D11.1 (K), D15.1 (K), D3.1 (K), D7.1 (K), J3.13 (Pin_13); no longer D13.1 (K), D14.1 (K), D5.1 (K), D6.1 (K), J3.4 (Pin_4)
- net ROW3: now also D12.1 (K), D4.1 (K), J3.15 (Pin_15); no longer D15.1 (K), D7.1 (K), J3.2 (Pin_2)
- net at J1.1 (Pin_1): now also D8.2 (A); no longer D15.2 (A)
- net at J1.11 (Pin_11): now also D3.2 (A); no longer D5.2 (A)
- net at J1.13 (Pin_13): now also D2.2 (A); no longer D3.2 (A)
- net at J1.3 (Pin_3): now also D7.2 (A); no longer D13.2 (A)
- net at J1.5 (Pin_5): now also D6.2 (A); no longer D11.2 (A)
- net at J1.7 (Pin_7): now also D5.2 (A); no longer D9.2 (A)
- net at J1.9 (Pin_9): now also D4.2 (A); no longer D7.2 (A)
- net at J2.11 (Pin_11): now also D11.2 (A); no longer D6.2 (A)
- net at J2.13 (Pin_13): now also D10.2 (A); no longer D4.2 (A)
- net at J2.15 (Pin_15): now also D9.2 (A); no longer D2.2 (A)
- net at J2.3 (Pin_3): now also D15.2 (A); no longer D14.2 (A)
- net at J2.5 (Pin_5): now also D14.2 (A); no longer D12.2 (A)
- net at J2.7 (Pin_7): now also D13.2 (A); no longer D10.2 (A)
- net at J2.9 (Pin_9): now also D12.2 (A); no longer D8.2 (A)
- new net +3.3V: J3.4 (Pin_4), U1.16 (V+)
- new net I2C-CLK: J3.6 (Pin_6)
- new net I2C-DAT: J3.8 (Pin_8)
- new net SPI-CIPO: J3.14 (Pin_14)
- new net SPI-CLK: J3.10 (Pin_10)
- new net SPI-COPI: J3.12 (Pin_12)
Other:
- note added: "Mounting Hole"
- moved on the sheet: D1, D10, D11, D12, D13, D14, D15, D16, D2, D3, D4, D5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
