File: PCB/Modules/Keymatrix/Keymatrix.kicad_pcb (KiCad board)
At the start: 2 copper layers, 30 x 64 mm, 54 parts, among them J1 In, J10 Col0, J11 Col1, J12 Col2, J13 Col3, J14 Col4, U1 74HC4051

Commit message: feat: LCD I2C interface.
Parts:
- moved G*** 20.6 mm to (46.4, 59.2)
Changed lines of the file:
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@@
 	(footprint "KTANE:KTANEIRL-0505"
 		(layer "F.Cu")
-		(at 64.8 49.95 90)
+		(at 46.3825 59.195 90)
 		(property "Reference" "G***"
 			(at 0 0 90)
@@
 	)
 	(gr_text "KTANE IRL by Melair\nKeymatrix (B01)"
-		(at 65.3 47.2 90)
+		(at 46.85875 56.81375 90)
 		(layer "F.SilkS")
 		(effects
