File: PCB/Modules/SPIRadioCFRTC/SPIRadioCFRTC.kicad_pcb (KiCad board)
At the start: 2 copper layers, 29 x 59 mm, 27 parts, among them J1 In, J2 Micro_SD_Card_Det_9pin, Q1 Q_NMOS_GSD, Q2 Q_NMOS_GSD, Q3 Q_NMOS_GSD, U1 DS1390U, U2 nRF24L01P_Module, U3 AMS1117-3.3, Y1 32.767kHz

Commit message: Convert all KiCad to 6.0, clean up libraries, remove files that shouldn't be committed.
Parts:
- BT1: footprint SPIRadioCFRTC:CellHolder -> KTANE:CellHolder
- J1: footprint Custom:PinHeader_2x08_P2.54mm_Vertical-Centered -> KTANE:PinHeader_2x08_P2.54mm_Vertical-Centered
- J2: footprint SPIRadioCFRTC:mSDCardSlot -> KTANE:mSDCardSlot
- U2: footprint SPIRadioCFRTC:NRF24L01P-Module -> KTANE:NRF24L01P-Module

Commit message: First pass of PCB rework.
Parts:
- removed C3: 10uF, Capacitor_SMD:C_0805_2012Metric
- removed Q1, Q2, Q3: Q_NMOS_GSD, Package_TO_SOT_SMD:SOT-23
- removed R10, R11, R2, R3, R4, R5, R6, R7, R8, R9: 10k, Resistor_SMD:R_0805_2012Metric
- removed REF**: MountingHole_3.2mm_M3, MountingHole:MountingHole_3.2mm_M3
- removed U3: AMS1117-3.3, Package_TO_SOT_SMD:SOT-23
- added C6: 10uF, Capacitor_SMD:C_0603_1608Metric, F.Cu at (47.5, 24.0)
- added C7: 0.1uF, Capacitor_SMD:C_0603_1608Metric, F.Cu at (47.5, 30.0)
- added H1: MountingHole, MountingHole:MountingHole_3.2mm_M3, F.Cu at (34.5, 75.0)
- added U4: ESP32-WROOM-32, RF_Module:ESP32-WROOM-32U, F.Cu at (39.4, 40.8)
- C1, C2: footprint Capacitor_SMD:C_0805_2012Metric -> Capacitor_SMD:C_0603_1608Metric
- C4: value 0.1uF -> 22uF; footprint Capacitor_SMD:C_0805_2012Metric -> Capacitor_SMD:C_0603_1608Metric
- C5: value 0.1uF -> 47uF; footprint Capacitor_SMD:C_0805_2012Metric -> Capacitor_SMD:C_0603_1608Metric
- J2: value Micro_SD_Card_Det_9pin -> ESP32; footprint KTANE:mSDCardSlot -> Connector:Tag-Connect_TC2030-IDC-NL_2x03_P1.27mm_Vertical
- R1: footprint Resistor_SMD:R_0805_2012Metric -> Resistor_SMD:R_0603_1608Metric
- moved C5 25.6 mm to (47.5, 27.0), turned to 0 degrees
- moved C4 24.1 mm to (47.5, 28.5), turned to 0 degrees
- moved J2 14.5 mm to (44.5, 52.5), turned to 180 degrees
- moved R1 10.1 mm to (47.5, 25.5), turned to 0 degrees
- moved C1 8.10 mm to (31.2, 52.5), turned to 0 degrees
- moved BT1 8.01 mm to (37.0, 63.0)
- moved U1 6.00 mm to (26.5, 54.0)
- moved Y1 6.00 mm to (22.0, 53.2)
- moved C2 3.10 mm to (25.0, 59.5)
- turned J1 to -90 degrees
Connections:
- C1 pad 1: +3V3 -> +3.3V
- C2 pad 1: +3V3 -> +3.3V
- C4 pad 1: +5V -> +3.3V
- C5 pad 1: +3V3 -> +3.3V
- J1 pad 1: GND -> RTC-CS
- J1 pad 10: NF24-CE -> SPI-CLK
- J1 pad 11: +5V -> ESP32-CS
- J1 pad 12: NF24-CS -> SPI-COPI
- J1 pad 13: +5V -> ESP32-RX
- J1 pad 14: SD-CS -> SPI-CIPO
- J1 pad 15: +5V -> ESP32-TX
- J1 pad 16: RTC-CS -> GND
- J1 pad 2: IN-MISO -> +5V
- J1 pad 3: GND -> RTC-INT
- J1 pad 4: IN-MOSI -> +3.3V
- J1 pad 5: GND -> NF24-CS
- J1 pad 6: IN-SCLK -> I2C-CLK
- J1 pad 7: GND -> NF24-CE
- J1 pad 8: INT -> I2C-DAT
- J1 pad 9: +5V -> NF24-INT
- J2 pad 1: unconnected-(J2-Pad1) -> ESP32-TX
- J2 pad 2: SD-CS -> +3.3V
- J2 pad 3: MOSI -> GND
- J2 pad 4: +3V3 -> EN
- J2 pad 5: SCLK -> ESP32-RX
- J2 pad 6: GND -> BOOT0
- R1 pad 1: IN-SCLK -> +3.3V
- R1 pad 2: +5V -> EN
- U1 pad 10: +3V3 -> +3.3V
- U1 pad 6: MOSI -> SPI-COPI
- U1 pad 7: MISO -> SPI-CIPO
- U1 pad 8: SCLK -> SPI-CLK
- U1 pad 9: INT -> RTC-INT
- U2 pad 1: +3V3 -> +3.3V
- U2 pad 4: SCLK -> SPI-CLK
- U2 pad 5: MOSI -> SPI-COPI
- U2 pad 6: MISO -> SPI-CIPO
- U2 pad 7: INT -> NF24-INT
Routing:
- net +3.3V: track 0.00 -> 88.6 mm, vias 0 -> 4
- net +3V3: track 73.0 -> 0.00 mm, vias 5 -> 0
- net SPI-COPI: track 0.00 -> 70.1 mm, vias 0 -> 3
- net INT: track 67.2 -> 0.00 mm, vias 5 -> 0
- net SPI-CLK: track 0.00 -> 63.6 mm, vias 0 -> 4
- net SPI-CIPO: track 0.00 -> 61.2 mm, vias 0 -> 2
- net MISO: track 60.4 -> 0.00 mm, vias 3 -> 0
- net MOSI: track 58.3 -> 0.00 mm, vias 5 -> 0
- net NF24-INT: track 0.00 -> 51.4 mm, vias 0 -> 1
- net SCLK: track 48.6 -> 0.00 mm, vias 3 -> 0
- net RTC-INT: track 0.00 -> 36.6 mm, vias 0 -> 1
- net EN: track 0.00 -> 34.6 mm, vias 0 -> 2
- net ESP32-CS: track 0.00 -> 33.9 mm, vias 0 -> 2
- net +5V: track 31.7 -> 0.00 mm
- net ESP32-TX: track 0.00 -> 29.4 mm, vias 0 -> 2
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Other:
- board text added: "Keep Talking and Nobody Explodes RTC/ESP32/nF24 Module (Rev B01)"
- board text removed: "Keep Talking and Nobody Explodes RTC/μSD/nF24 Module (Rev A02)"
