File: PCB/Others/2FALCD/2FALCD.kicad_pcb (KiCad board)
At the start: 2 copper layers, 65 x 20 mm, 15 parts, among them J2 VCC, J3 /INT, J4 SDA, J5 SCL, J6 VLCD, J7 GND, SW1 Interact, U1 HT16C21A-28

Commit message: Include all corrections, mint new gerbers. Update some to KiCad 10.
Other:
- board text added: "KTANE IRL by Melair 2FA LCD (A02)"
- board text removed: "KTANE IRL by Melair 2FA LCD (A01)"
