File: PCB/Others/2FALCD/2FALCD.kicad_sch (KiCad schematic)
At the start: 14 parts, among them J2 VCC, J3 /INT, J4 SDA, J5 SCL, J6 VLCD, J7 GND, SW1 Interact, U1 HT16C21A-28

Commit message: Include all corrections, mint new gerbers. Update some to KiCad 10.
Parts:
- DS1: value ~ -> (none)
Connections:
- no-connect marks 2 -> 8
