File: PCB/Modules/Power/Power.kicad_sch (KiCad schematic)
At the start: 12 parts, among them J1 Out1, J10 Comms, J11 Battery, J12 Comms, J2 Out2, J3 USB_C_Receptacle_USB2.0_14P, J4 VBus, J5 VBus, J6 Comms, J7 Comms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

Commit message: Update to KiCad 10.
Connections:
- net Battery/GND is gone; now on net Battery/GND: J11.1 (Pin_1)
- net Interface/CC1 is gone; now on net Interface/CC1: J6.1 (Pin_1)
- net Interface/CC2 is gone; now on net Interface/CC2: J6.2 (Pin_2)
- net Interface/D+ is gone; now on net Interface/D+: J6.4 (Pin_4)
- net Interface/D- is gone; now on net Interface/D-: J6.3 (Pin_3)
- net Interface/GND is gone; now on net Interface/GND: J4.1 (Pin_1)
- net Interface/VBUS is gone; now on net Interface/VBUS: J4.2 (Pin_2)
- net Manager/GND is gone; now on net Manager/GND: J1.1 (Pin_1)
- net Battery/GND: no longer J12.5 (Pin_5)
- net Interface/CC1: no longer J3.A5 (CC1)
- net Interface/CC2: no longer J3.B5 (CC2)
- net Interface/D+: no longer J3.A6 (D+), J3.B6 (D+)
- net Interface/D-: no longer J3.A7 (D-), J3.B7 (D-)
- net Interface/GND: no longer J3.A1 (GND), J3.A12 (GND), J3.B1 (GND), J3.B12 (GND)
- net Interface/VBUS: no longer J3.A4 (VBUS), J3.A9 (VBUS), J3.B4 (VBUS), J3.B9 (VBUS)
- net Manager/GND: no longer J5.1 (Pin_1)
- new net Battery/GND: J12.5 (Pin_5)
- new net Interface/CC1: J3.A5 (CC1)
- new net Interface/CC2: J3.B5 (CC2)
- new net Interface/D+: J3.A6 (D+), J3.B6 (D+)
- new net Interface/D-: J3.A7 (D-), J3.B7 (D-)
- new net Interface/GND: J3.A1 (GND), J3.A12 (GND), J3.B1 (GND), J3.B12 (GND)
- new net Interface/VBUS: J3.A4 (VBUS), J3.A9 (VBUS), J3.B4 (VBUS), J3.B9 (VBUS)
- new net Manager/GND: J5.1 (Pin_1)
