File: PCB/Modules/Power/manager.kicad_sch (KiCad schematic)
At the start: 99 parts, among them J13 ICSP, Q1 NMOS, Q2 Q_NMOS, Q3 Q_NMOS, Q4 Q_NMOS, Q5 Q_NMOS, Q6 NMOS, Q7 NMOS, Q8 Q_NMOS_GSD, U1 PIC18F15Q40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

Commit message: Update to KiCad 10.
Parts:
- D4, D5, D7, D8: value ~ -> (none)
