File: PCB/Modules/Audio/Audio.kicad_pcb (KiCad board)
At the start: 4 copper layers, 80 x 50 mm, 65 parts, among them J1 ESP32, J2 Control Board, J3 VBUS, J4 RIGHT, J5 LEFT, Q1 Q_NMOS_GSD, Q2 Q_PMOS_GSD, SW1 RUN/~{PROG}, U1 Audio, U2 TAS5733

Commit message: feat: Update audio board to consume I2S from STM32 parent board, removing ESP32.
Parts:
- removed C1: 22uF, Capacitor_SMD:C_1206_3216Metric
- removed C2: 47uF, Capacitor_SMD:C_0603_1608Metric
- removed C3: 10uF, Capacitor_SMD:C_0603_1608Metric
- removed C4: 0.1uF, Capacitor_SMD:C_0603_1608Metric
- removed J1: ESP32, Connector:Tag-Connect_TC2030-IDC-NL_2x03_P1.27mm_Vertical
- removed R1, R2: 10k, Resistor_SMD:R_0603_1608Metric
- removed R6, R7: 4.7k, Resistor_SMD:R_0603_1608Metric
- removed SW1: RUN/~{PROG}, KTANE:JS102011JCQN
- removed U1: Audio, KTANE:ESP32-C5-WROOM-1U
- H1, H2, H3, H4: footprint MountingHole:MountingHole_3.2mm_M3 -> KTANE:MountingHole_3.2mm_M3_NoCopper
- J4: value RIGHT -> AB
- J5: value LEFT -> CD
- moved R5 20.7 mm to (68.6, 60.3), turned to 180 degrees
- moved J2 17.9 mm to (61.6, 56.5), turned to 0 degrees
- moved R3 16.3 mm to (68.6, 65.4), turned to 180 degrees
- moved R9 13.5 mm to (68.6, 47.6), turned to 180 degrees
- moved R12 12.8 mm to (68.6, 50.2), turned to 180 degrees
- moved R4 12.7 mm to (68.6, 52.7), turned to 180 degrees
- moved R8 8.80 mm to (68.6, 55.2), turned to 180 degrees
Connections:
- J2 pad 1: HOST-SPI-CIPO -> unconnected-(J2-SPI-CIPO-Pad1)
- J2 pad 10: ~{HOST-SPI-CS} -> unconnected-(J2-I4-Pad10)
- J2 pad 12: ESP32-EN -> /~{FAULT}
- J2 pad 14: unconnected-(J2-I1-Pad14) -> /AUDIO_PVDD_ON
- J2 pad 16: unconnected-(J2-I0-Pad16) -> /~{RST}
- J2 pad 2: unconnected-(J2-I7-Pad2) -> /LRCLK
- J2 pad 3: HOST-SPI-CLK -> unconnected-(J2-SPI-CLK-Pad3)
- J2 pad 4: unconnected-(J2-I6-Pad4) -> /SCLK
- J2 pad 5: HOST-SPI-COPI -> unconnected-(J2-SPI-COPI-Pad5)
- J2 pad 6: unconnected-(J2-I5-Pad6) -> /~{PDN}
- J2 pad 7: unconnected-(J2-SDA-Pad7) -> /SDA
- J2 pad 8: ~{HOST-INT} -> /SDIN
- J2 pad 9: unconnected-(J2-SCL-Pad9) -> /SCL
Routing:
- net ESP32-EN: track 41.1 -> 0.00 mm
- net BOOT0: track 33.4 -> 0.00 mm, vias 2 -> 0
- net /~{FAULT}: track 23.7 -> 54.5 mm
- net /~{PDN}: track 14.6 -> 39.5 mm
- net ~{HOST-SPI-CS}: track 20.3 -> 0.00 mm
- net ~{HOST-INT}: track 16.8 -> 0.00 mm
- net /LRCLK: track 12.3 -> 26.5 mm
- net ESP32-PROG-TX: track 14.0 -> 0.00 mm, vias 2 -> 0
- net ESP32-PROG-RX: track 11.2 -> 0.00 mm
- net HOST-SPI-CIPO: track 11.1 -> 0.00 mm
- net HOST-SPI-COPI: track 11.0 -> 0.00 mm
- net /SCLK: track 14.2 -> 25.1 mm
- net HOST-SPI-CLK: track 10.5 -> 0.00 mm
- net +3.3V: track 23.5 -> 13.1 mm, vias 7 -> 2
- net /AUDIO_PVDD_ON: track 40.9 -> 50.7 mm, vias 2 -> 0
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Other:
- board text added: "KTANE IRL by Melair Audio (C01)"
- board text removed: "KTANE IRL by Melair Audio (B01)"
