File: PCB/Modules/Audio/Audio.kicad_sch (KiCad schematic)
At the start: 64 parts, among them J1 ESP32, J2 Control Board, J3 VBUS, J4 RIGHT, J5 LEFT, Q1 Q_NMOS_GSD, Q2 Q_PMOS_GSD, SW1 RUN/~{PROG}, U1 Audio, U2 TAS5733

Commit message: feat: Update audio board to consume I2S from STM32 parent board, removing ESP32.
Parts:
- removed C1: 22uF, Capacitor_SMD:C_1206_3216Metric, symbol Device:C_Small
- removed C2: 47uF, Capacitor_SMD:C_0603_1608Metric, symbol Device:C_Small
- removed C3: 10uF, Capacitor_SMD:C_0603_1608Metric, symbol Device:C_Small
- removed C4: 0.1uF, Capacitor_SMD:C_0603_1608Metric, symbol Device:C_Small
- removed J1: ESP32, Connector:Tag-Connect_TC2030-IDC-NL_2x03_P1.27mm_Vertical, symbol Connector_Generic:Conn_02x03_Odd_Even
- removed R1, R2: 10k, Resistor_SMD:R_0603_1608Metric, symbol Device:R_Small
- removed R6, R7: 4.7k, Resistor_SMD:R_0603_1608Metric, symbol Device:R_Small
- removed SW1: RUN/~{PROG}, KTANE:JS102011JCQN, symbol Switch:SW_SPDT
- removed U1: Audio, KTANE:ESP32-C5-WROOM-1U, symbol KTANE:ESP32-C5-WROOM-1U
- H1, H2, H3, H4: footprint MountingHole:MountingHole_3.2mm_M3 -> KTANE:MountingHole_3.2mm_M3_NoCopper
- J4: value RIGHT -> AB
- J5: value LEFT -> CD
Connections:
- net ESP32-EN is gone; now on net ~{FAULT}: J2.12 (I5)
- net ~{HOST-INT} is gone; now on net SDIN: J2.8 (I3)
- net AUDIO_PVDD_ON: now also J2.14 (I6)
- net LRCLK: now also J2.2 (I0)
- net SCL: now also J2.9 (SCL)
- net SCLK: now also J2.4 (I1)
- net SDA: now also J2.7 (SDA)
- net ~{PDN}: now also J2.6 (I2)
- net ~{RST}: now also J2.16 (I7)
- net HOST-SPI-CIPO: no longer names the net of J2.1 (SPI-CIPO)
- net HOST-SPI-CLK: no longer names the net of J2.3 (SPI-CLK)
- net HOST-SPI-COPI: no longer names the net of J2.5 (SPI-COPI)
- net ~{HOST-SPI-CS}: no longer names the net of J2.10 (I4)
- no-connect marks 15 -> 6
Other:
- note removed: "Used for SPI PSRAM /CS."
- moved on the sheet: J2

Commit message: feat: Export new revision BOM, allow in .gitignore, fix up revisions in schematics.
Other:
- title: (none) -> KTANE - Audio Board
Changed lines of the file:
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@@
 	(generator_version "10.0")
 	(paper "A3")
+	(title_block
+		(title "KTANE - Audio Board")
+		(rev "C01")
+	)
 	(rectangle
 		(start 30.48 215.9)
