File: PCB/Others/Strikes/Strikes.kicad_pcb (KiCad board)
At the start: 2 copper layers, 54 x 35 mm, 25 parts, among them J1 3V3, J2 LAT, J3 SCLK, J4 SIN, J5 BLANK, J6 SCL, J7 SDA, J8 GND, U1 AD5272BRMZ-50, U2 TLC59281, U3 AD5272BRMZ-50, U4 TLC59281

Commit message: fix: Labels on Strikes PCB for SDA/SCL are swapped.
Parts:
- J6: value SCL -> SDA
- J7: value SDA -> SCL
