File: PCB/Modules/Comms/Comms.kicad_sch (KiCad schematic)
At the start: 50 parts, among them J1 In, J10 1PPS In, J11 32MHz Out, J12 Shield, J13 Shield, J2 Test, J3 Bus, J4 Bus, J5 SWD, J6 Shield, J7 Shield, J8 Shield, J9 Shield, Q1 Q_PMOS_GSD, U1 STM32WB09KEVx, U2 THVD1420D, U3 MLPF-NRG-01D3, Y1 32MHz, Y2 32.768k

Commit message: feat: Version C02 of the comms board, fixing errors found during testing.
Parts:
- removed J11: 32MHz Out, Connector_Coaxial:U.FL_Hirose_U.FL-R-SMT-1_Vertical, symbol KTANE:UFLConnector
- removed JP1: NO BATT, Jumper:SolderJumper-2_P1.3mm_Open_Pad1.0x1.5mm, symbol Jumper:Jumper_2_Open
- added C31, C9: 0.1μF, Capacitor_SMD:C_0603_1608Metric, symbol Device:C_Small
- added C32: 4.7uF, Capacitor_SMD:C_0603_1608Metric, symbol Device:C_Small
- added D3: Status, LED_SMD:LED_0603_1608Metric, symbol Device:LED
- added J14: UART, Connector:Tag-Connect_TC2030-IDC-NL_2x03_P1.27mm_Vertical, symbol Connector_Generic:Conn_02x03_Odd_Even
- added L1: 10uH, Inductor_SMD:L_0805_2012Metric, symbol Device:L_Small
- added L2: 22nH, Inductor_SMD:L_0402_1005Metric, symbol Device:L_Small
- added R10, R12, R9: 10k, Resistor_SMD:R_0603_1608Metric, symbol Device:R_Small
- added R11: 51, Resistor_SMD:R_0603_1608Metric, symbol Device:R_Small
- added SW1: Boot, KTANE:PTS526Sx15SMTR2xLFS, symbol KTANE:SW_Push_4Pin
- J10: value 1PPS In -> 1PPS
- J2: value Test -> ANT
- U1: symbol MCU_ST_STM32WB:STM32WB09KEVx -> KTANE:STM32WB09KEVx
Connections:
- net +3.3V: now also U1.1 (PB3); no longer U1.4 (PB0)
- net +3.3VP: now also D3.2 (A), R9.1, SW1.3; no longer U1.27 (VFBSD)
- net GND: now also U1.33 (VSSSD), C31.2, C32.2, C9.2, J14.5 (Pin_5), R10.1, R12.2
- net ~{BLE_INT}: now also J1.2 (I0); no longer J1.10 (I4)
- net ~{RUN}: now also J1.16 (I7), U1.18 (PB15), R9.2; no longer U1.30 (PB5)
- net at U1.11 (PA10): now also R10.2
- net at U1.25 (VLXSD): now also L2.2
- net BUTTON: now reaches U1.3 (PB1)
- net BUTTON: now also C9.1, R12.1, SW1.1
- net CAL_OUT: no longer names the net of U1.19 (PB14)
- net SCL: no longer names the net of U1.8 (PA0)
- net SCL: no longer J1.9 (SCL)
- net SDA: no longer names the net of U1.7 (PA1)
- net SDA: no longer J1.7 (SDA)
- net SPI-CIPO: no longer names the net of J1.1 (SPI-CIPO)
- net SPI-CIPO: no longer U1.9 (PA8)
- net SPI-CLK: no longer names the net of J1.3 (SPI-CLK)
- net SPI-CLK: no longer U1.1 (PB3)
- net SPI-COPI: no longer names the net of U1.12 (PA11)
- net SPI-COPI: no longer J1.5 (SPI-COPI)
- net ~{SPI-CS} renamed DEBUG_TX
- net DEBUG_TX: now also J14.3 (Pin_3); no longer J1.2 (I0)
- new net: C31.1, C32.1, L1.1, U1.27 (VFBSD)
- new net: L1.2, L2.1
- new net: D3.1 (K), R11.1
- new net DEBUG_RX: J14.4 (Pin_4), U1.9 (PA8)
- new net STATUS: R11.2, U1.4 (PB0)
- no-connect marks 7 -> 18
Other:
- note added: "STM32WB09"
- note added: "Serial Debug"
- note removed: "ESP32"
- moved on the sheet: BT1
