File: PCB/Modules/LocalAudio/LocalAudio.kicad_pcb (KiCad board)
At the start: 4 copper layers, 30 x 64 mm, 24 parts, among them J1 In, J2 Speaker, J3 Headphones, J4 Volume, U1 TLV320DAC32

Commit message: feat: Missing commit.
Parts:
- moved G*** 31.9 mm to (22.3, 78.3)
Routing:
- net I2C-DAT: track 32.8 -> 33.5 mm
- net GND: vias 1 -> 43
